File: Irrigation_IoT/Irrigation_IoT.kicad_pcb (KiCad board)
At the start: 2 copper layers, 99.8 x 60.2 mm, 79 parts, among them IC1 ESP32-S3-WROOM-1-N16R8, IC2 CP2102-GM, J1 Barrel_Jack_MountingPin, J10 Conn_12V, J2 USB_B_Micro, J3 Screw_Terminal_01x03, J4 I2C Extern, J5 Connector DHT22, J6 Connector Display, J7 Screw_Terminal_01x03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

Commit message: Inclusão do step
Parts:
- J6: footprint Connector_PinSocket_2.54mm:PinSocket_1x04_P2.54mm_Vertical -> Connector_PinSocket_2.54mm:PinSocket_1x04_P2.54mm_Vertical_DISPLAY_OLED
Connections:
- R9 pad 1: Net-(Q3-B) -> Net-(R8-Pad2)

Commit message: atualização de arquivos
Routing:
- net Earth: vias 75 -> 94
Other:
- board text added: "RavaBoard_IoT v1.1"
- board text removed: "RavaBorad_IoT v1.0"
