File: Irrigation_IoT/Irrigation_IoT.kicad_sch (KiCad schematic)
At the start: 46 parts, among them IC1 ESP32-S3-WROOM-1-N16R8, IC2 CP2102-GM, J1 Barrel_Jack_MountingPin, J2 USB_B_Micro, J4 I2C Extern, J5 Connector DHT22, J6 Connector Display, Q1 BC817, Q2 BC817, SW1 SW_MEC_5G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

Commit message: atualização de arquivos
Parts:
- J6: footprint Connector_PinSocket_2.54mm:PinSocket_1x04_P2.54mm_Vertical -> Connector_PinSocket_2.54mm:PinSocket_1x04_P2.54mm_Vertical_DISPLAY_OLED
Changed lines of the file:
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@@
 			)
 		)
-		(property "Footprint" "Connector_PinSocket_2.54mm:PinSocket_1x04_P2.54mm_Vertical"
+		(property "Footprint" "Connector_PinSocket_2.54mm:PinSocket_1x04_P2.54mm_Vertical_DISPLAY_OLED"
 			(at 142.621 32.766 0)
 			(effects
@@
 			)
 		)
-		(property "Description" ""
+		(property "Description" "Generic connector, single row, 01x04, script generated"
 			(at 142.621 32.766 0)
 			(effects
