File: Irrigation_IoT/Rele.kicad_sch (KiCad schematic)
At the start: 27 parts, among them J16 Conn_12V, J17 Conn_12V, J3 Screw_Terminal_01x03, J7 Screw_Terminal_01x03, J8 Screw_Terminal_01x02, K1 AX1RC2, K2 AX1RC2, Q1 BC817, Q2 BC817, U3 PC817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

Commit message: atualização de arquivos
Parts:
- removed LED2, LED3: LED_VM, LED_THT:LED_D3.0mm, symbol Device:LED
- removed R8: 10K, Resistor_SMD:R_0805_2012Metric, symbol Device:R
Connections:
- net Earth: now also U3.2, U4.2
Other:
- note added: "Verificar funcionabilidade"
- note removed: "Altamente problemático"
- moved on the sheet: Q2, R4, R5, U3
